Commit message: Add inertial properties to each link of IRB4600 60/20.5

File: abb_irb4600_support/urdf/irb4600_60_205_macro.urdf.xacro (robot description, xacro)
@@ -17,4 +17,12 @@
         </material>
       </visual>
+      <!-- The following are estimates only, as computed using total robot mass of 445kg distributed according to link volumes. -->
+      <inertial>
+        <mass value="81.828765"/>
+        <inertia ixx="1.1415" ixy="0.0105902" ixz="0.156701"
+                 iyy="2.31965" iyz="0.00032"
+                 izz="3.13136"/>
+        <origin xyz="-0.0914 0.000381 0.08247" rpy="0 0 0"/>
+      </inertial>
     </link>
     <link name="${prefix}link_1">
@@ -30,4 +38,12 @@
         <material name="yellow"/>
       </visual>
+      <!-- The following are estimates only, as computed using total robot mass of 445kg distributed according to link volumes. -->
+      <inertial>
+        <mass value="114.303365"/>
+        <inertia ixx="2.99197" ixy="-0.262121" ixz="0.0804318"
+                 iyy="3.89993" iyz="-0.279368"
+                 izz="3.12186"/>
+        <origin xyz="0.076986 0.024762 -0.0947" rpy="0 0 0"/>
+      </inertial>
     </link>
     <link name="${prefix}link_2">
@@ -43,4 +59,12 @@
         <material name="yellow"/>
       </visual>
+      <!-- The following are estimates only, as computed using total robot mass of 445kg distributed according to link volumes. -->
+      <inertial>
+        <mass value="75.83976"/>
+        <inertia ixx="5.85548" ixy="-0.00008" ixz="0.000798"
+                 iyy="6.06764" iyz="0.198884"
+                 izz="0.434182"/>
+        <origin xyz="0 -0.17055 0.396832" rpy="0 0 0"/>
+      </inertial>
     </link>
     <link name="${prefix}link_3">
@@ -56,4 +80,12 @@
         <material name="yellow"/>
       </visual>
+      <!-- The following are estimates only, as computed using total robot mass of 445kg distributed according to link volumes. -->
+      <inertial>
+        <mass value="128.2082"/>
+        <inertia ixx="3.06222" ixy="0.199317" ixz="-0.309802"
+                 iyy="3.76188" iyz="0.0384368"
+                 izz="3.09117"/>
+        <origin xyz="0.040168 0.0493055 0.119626" rpy="0 0 0"/>
+      </inertial>
     </link>
     <link name="${prefix}link_4">
@@ -69,4 +101,12 @@
         <material name="yellow"/>
       </visual>
+      <!-- The following are estimates only, as computed using total robot mass of 445kg distributed according to link volumes. -->
+      <inertial>
+        <mass value="30.039968"/>
+        <inertia ixx="0.143877" ixy="0.0152815" ixz="0.00617976"
+                 iyy="1.24666" iyz="0.00008"
+                 izz="1.29441"/>
+        <origin xyz="0.733488 -0.0019699 -0.002854" rpy="0 0 0"/>
+      </inertial>
     </link>
     <link name="${prefix}link_5">
@@ -82,4 +122,12 @@
         <material name="yellow"/>
       </visual>
+      <!-- The following are estimates only, as computed using total robot mass of 445kg distributed according to link volumes. -->
+      <inertial>
+        <mass value="4.06033"/>
+        <inertia ixx="0.00817067" ixy="0.0" ixz="-0.00005"
+                 iyy="0.00847828" iyz="0.00001"
+                 izz="0.009"/>
+        <origin xyz="-0.001046 -0.003447 0.000404" rpy="0 0 0"/>
+      </inertial>
     </link>
     <link name="${prefix}link_6">
@@ -95,4 +143,12 @@
         <material name="yellow"/>
       </visual>
+      <!-- The following are estimates only, as computed using total robot mass of 445kg distributed according to link volumes. -->
+      <inertial>
+        <mass value="0.71955"/>
+        <inertia ixx="0.00101673" ixy="0.0" ixz="0.0"
+                 iyy="0.000771006" iyz="0.0"
+                 izz="0.000776247"/>
+        <origin xyz="-0.0216378 -0.000286 0.000136" rpy="0 0 0"/>
+      </inertial>
     </link>
     <!-- end of link list -->

Commit message: update xacro

File: abb_irb4600_support/urdf/irb4600_60_205_macro.urdf.xacro (robot description, xacro)
@@ -6,22 +6,23 @@
       <collision name="collision">
         <geometry>
-          <mesh filename="package://abb_irb4600_support/meshes/irb4600/collision/base_link.stl"/>
-        </geometry>
-      </collision>
-      <visual name="visual">
-        <geometry>
-          <mesh filename="package://abb_irb4600_support/meshes/irb4600/visual/base_link.dae"/>
+          <mesh filename="package://abb_irb4600_support/meshes/irb4600/collision/base_link.stl" />
+        </geometry>
+      </collision>
+      <visual name="visual">
+        <geometry>
+          <mesh filename="package://abb_irb4600_support/meshes/irb4600/visual_obj/base_link.obj" />
         </geometry>
         <material name="yellow">
-          <color rgba="1 1 0 1"/>
+          <color rgba="1 1 0 1" />
         </material>
       </visual>
-      <!-- The following are estimates only, as computed using total robot mass of 445kg distributed according to link volumes. -->
-      <inertial>
-        <mass value="81.828765"/>
+      <!-- The following are estimates only, as computed using total robot mass of 445kg distributed
+      according to link volumes. -->
+      <inertial>
+        <mass value="81.828765" />
         <inertia ixx="1.1415" ixy="0.0105902" ixz="0.156701"
-                 iyy="2.31965" iyz="0.00032"
-                 izz="3.13136"/>
-        <origin xyz="-0.0914 0.000381 0.08247" rpy="0 0 0"/>
+          iyy="2.31965" iyz="0.00032"
+          izz="3.13136" />
+        <origin xyz="-0.0914 0.000381 0.08247" rpy="0 0 0" />
       </inertial>
     </link>
@@ -29,20 +30,21 @@
       <collision name="collision">
         <geometry>
-          <mesh filename="package://abb_irb4600_support/meshes/irb4600/collision/link_1.stl"/>
-        </geometry>
-      </collision>
-      <visual name="visual">
-        <geometry>
-          <mesh filename="package://abb_irb4600_support/meshes/irb4600/visual/link_1.dae"/>
-        </geometry>
-        <material name="yellow"/>
-      </visual>
-      <!-- The following are estimates only, as computed using total robot mass of 445kg distributed according to link volumes. -->
-      <inertial>
-        <mass value="114.303365"/>
+          <mesh filename="package://abb_irb4600_support/meshes/irb4600/collision/link_1.stl" />
+        </geometry>
+      </collision>
+      <visual name="visual">
+        <geometry>
+          <mesh filename="package://abb_irb4600_support/meshes/irb4600/visual_obj/link_1.obj" />
+        </geometry>
+        <material name="yellow" />
+      </visual>
+      <!-- The following are estimates only, as computed using total robot mass of 445kg distributed
+      according to link volumes. -->
+      <inertial>
+        <mass value="114.303365" />
         <inertia ixx="2.99197" ixy="-0.262121" ixz="0.0804318"
-                 iyy="3.89993" iyz="-0.279368"
-                 izz="3.12186"/>
-        <origin xyz="0.076986 0.024762 -0.0947" rpy="0 0 0"/>
+          iyy="3.89993" iyz="-0.279368"
+          izz="3.12186" />
+        <origin xyz="0.076986 0.024762 -0.0947" rpy="0 0 0" />
       </inertial>
     </link>
@@ -50,20 +52,21 @@
       <collision name="collision">
         <geometry>
-          <mesh filename="package://abb_irb4600_support/meshes/irb4600_60_205/collision/link_2.stl"/>
-        </geometry>
-      </collision>
-      <visual name="visual">
-        <geometry>
-          <mesh filename="package://abb_irb4600_support/meshes/irb4600_60_205/visual/link_2.dae"/>
-        </geometry>
-        <material name="yellow"/>
-      </visual>
-      <!-- The following are estimates only, as computed using total robot mass of 445kg distributed according to link volumes. -->
-      <inertial>
-        <mass value="75.83976"/>
+          <mesh filename="package://abb_irb4600_support/meshes/irb4600_60_205/collision/link_2.stl" />
+        </geometry>
+      </collision>
+      <visual name="visual">
+        <geometry>
+          <mesh filename="package://abb_irb4600_support/meshes/irb4600_60_205/visual_obj/link_2.obj" />
+        </geometry>
+        <material name="yellow" />
+      </visual>
+      <!-- The following are estimates only, as computed using total robot mass of 445kg distributed
+      according to link volumes. -->
+      <inertial>
+        <mass value="75.83976" />
         <inertia ixx="5.85548" ixy="-0.00008" ixz="0.000798"
-                 iyy="6.06764" iyz="0.198884"
-                 izz="0.434182"/>
-        <origin xyz="0 -0.17055 0.396832" rpy="0 0 0"/>
+          iyy="6.06764" iyz="0.198884"
+          izz="0.434182" />
+        <origin xyz="0 -0.17055 0.396832" rpy="0 0 0" />
       </inertial>
     </link>
@@ -71,20 +74,21 @@
       <collision name="collision">
         <geometry>
-          <mesh filename="package://abb_irb4600_support/meshes/irb4600_60_205/collision/link_3.stl"/>
-        </geometry>
-      </collision>
-      <visual name="visual">
-        <geometry>
-          <mesh filename="package://abb_irb4600_support/meshes/irb4600_60_205/visual/link_3.dae"/>
-        </geometry>
-        <material name="yellow"/>
-      </visual>
-      <!-- The following are estimates only, as computed using total robot mass of 445kg distributed according to link volumes. -->
-      <inertial>
-        <mass value="128.2082"/>
+          <mesh filename="package://abb_irb4600_support/meshes/irb4600_60_205/collision/link_3.stl" />
+        </geometry>
+      </collision>
+      <visual name="visual">
+        <geometry>
+          <mesh filename="package://abb_irb4600_support/meshes/irb4600_60_205/visual_obj/link_3.obj" />
+        </geometry>
+        <material name="yellow" />
+      </visual>
+      <!-- The following are estimates only, as computed using total robot mass of 445kg distributed
+      according to link volumes. -->
+      <inertial>
+        <mass value="128.2082" />
         <inertia ixx="3.06222" ixy="0.199317" ixz="-0.309802"
-                 iyy="3.76188" iyz="0.0384368"
-                 izz="3.09117"/>
-        <origin xyz="0.040168 0.0493055 0.119626" rpy="0 0 0"/>
+          iyy="3.76188" iyz="0.0384368"
+          izz="3.09117" />
+        <origin xyz="0.040168 0.0493055 0.119626" rpy="0 0 0" />
       </inertial>
     </link>
@@ -92,20 +96,21 @@
       <collision name="collision">
         <geometry>
-          <mesh filename="package://abb_irb4600_support/meshes/irb4600_60_205/collision/link_4.stl"/>
-        </geometry>
-      </collision>
-      <visual name="visual">
-        <geometry>
-          <mesh filename="package://abb_irb4600_support/meshes/irb4600_60_205/visual/link_4.dae"/>
-        </geometry>
-        <material name="yellow"/>
-      </visual>
-      <!-- The following are estimates only, as computed using total robot mass of 445kg distributed according to link volumes. -->
-      <inertial>
-        <mass value="30.039968"/>
+          <mesh filename="package://abb_irb4600_support/meshes/irb4600_60_205/collision/link_4.stl" />
+        </geometry>
+      </collision>
+      <visual name="visual">
+        <geometry>
+          <mesh filename="package://abb_irb4600_support/meshes/irb4600_60_205/visual_obj/link_4.obj" />
+        </geometry>
+        <material name="yellow" />
+      </visual>
+      <!-- The following are estimates only, as computed using total robot mass of 445kg distributed
+      according to link volumes. -->
+      <inertial>
+        <mass value="30.039968" />
         <inertia ixx="0.143877" ixy="0.0152815" ixz="0.00617976"
-                 iyy="1.24666" iyz="0.00008"
-                 izz="1.29441"/>
-        <origin xyz="0.733488 -0.0019699 -0.002854" rpy="0 0 0"/>
+          iyy="1.24666" iyz="0.00008"
+          izz="1.29441" />
+        <origin xyz="0.733488 -0.0019699 -0.002854" rpy="0 0 0" />
       </inertial>
     </link>
@@ -113,20 +118,21 @@
       <collision name="collision">
         <geometry>
-          <mesh filename="package://abb_irb4600_support/meshes/irb4600_60_205/collision/link_5.stl"/>
-        </geometry>
-      </collision>
-      <visual name="visual">
-        <geometry>
-          <mesh filename="package://abb_irb4600_support/meshes/irb4600_60_205/visual/link_5.dae"/>
-        </geometry>
-        <material name="yellow"/>
-      </visual>
-      <!-- The following are estimates only, as computed using total robot mass of 445kg distributed according to link volumes. -->
-      <inertial>
-        <mass value="4.06033"/>
+          <mesh filename="package://abb_irb4600_support/meshes/irb4600_60_205/collision/link_5.stl" />
+        </geometry>
+      </collision>
+      <visual name="visual">
+        <geometry>
+          <mesh filename="package://abb_irb4600_support/meshes/irb4600_60_205/visual_obj/link_5.obj" />
+        </geometry>
+        <material name="yellow" />
+      </visual>
+      <!-- The following are estimates only, as computed using total robot mass of 445kg distributed
+      according to link volumes. -->
+      <inertial>
+        <mass value="4.06033" />
         <inertia ixx="0.00817067" ixy="0.0" ixz="-0.00005"
-                 iyy="0.00847828" iyz="0.00001"
-                 izz="0.009"/>
-        <origin xyz="-0.001046 -0.003447 0.000404" rpy="0 0 0"/>
+          iyy="0.00847828" iyz="0.00001"
+          izz="0.009" />
+        <origin xyz="-0.001046 -0.003447 0.000404" rpy="0 0 0" />
       </inertial>
     </link>
@@ -134,20 +140,21 @@
       <collision name="collision">
         <geometry>
-          <mesh filename="package://abb_irb4600_support/meshes/irb4600_60_205/collision/link_6.stl"/>
-        </geometry>
-      </collision>
-      <visual name="visual">
-        <geometry>
-          <mesh filename="package://abb_irb4600_support/meshes/irb4600_60_205/visual/link_6.dae"/>
-        </geometry>
-        <material name="yellow"/>
-      </visual>
-      <!-- The following are estimates only, as computed using total robot mass of 445kg distributed according to link volumes. -->
-      <inertial>
-        <mass value="0.71955"/>
+          <mesh filename="package://abb_irb4600_support/meshes/irb4600_60_205/collision/link_6.stl" />
+        </geometry>
+      </collision>
+      <visual name="visual">
+        <geometry>
+          <mesh filename="package://abb_irb4600_support/meshes/irb4600_60_205/visual_obj/link_6.obj" />
+        </geometry>
+        <material name="yellow" />
+      </visual>
+      <!-- The following are estimates only, as computed using total robot mass of 445kg distributed
+      according to link volumes. -->
+      <inertial>
+        <mass value="0.71955" />
         <inertia ixx="0.00101673" ixy="0.0" ixz="0.0"
-                 iyy="0.000771006" iyz="0.0"
-                 izz="0.000776247"/>
-        <origin xyz="-0.0216378 -0.000286 0.000136" rpy="0 0 0"/>
+          iyy="0.000771006" iyz="0.0"
+          izz="0.000776247" />
+        <origin xyz="-0.0216378 -0.000286 0.000136" rpy="0 0 0" />
       </inertial>
     </link>
@@ -155,44 +162,44 @@
     <!-- joint list -->
     <joint type="revolute" name="${prefix}joint_1">
-      <origin xyz="0 0 0.495" rpy="0 0 0"/>
-      <axis xyz="0 0 1"/>
-      <parent link="${prefix}base_link"/>
-      <child link="${prefix}link_1"/>
-      <limit effort="0" lower="-3.141" upper="3.141" velocity="3.054"/>
+      <origin xyz="0 0 0.495" rpy="0 0 0" />
+      <axis xyz="0 0 1" />
+      <parent link="${prefix}base_link" />
+      <child link="${prefix}link_1" />
+      <limit effort="0" lower="-3.141" upper="3.141" velocity="3.054" />
     </joint>
     <joint type="revolute" name="${prefix}joint_2">
-      <origin xyz="0.175 0 0" rpy="0 0 0"/>
-      <axis xyz="0 1 0"/>
-      <parent link="${prefix}link_1"/>
-      <child link="${prefix}link_2"/>
-      <limit effort="0" lower="-1.570" upper="2.617" velocity="3.054"/>
+      <origin xyz="0.175 0 0" rpy="0 0 0" />
+      <axis xyz="0 1 0" />
+      <parent link="${prefix}link_1" />
+      <child link="${prefix}link_2" />
+      <limit effort="0" lower="-1.570" upper="2.617" velocity="3.054" />
     </joint>
     <joint type="revolute" name="${prefix}joint_3">
-      <origin xyz="0 0 0.9" rpy="0 0 0"/>
-      <axis xyz="0 1 0"/>
-      <parent link="${prefix}link_2"/>
-      <child link="${prefix}link_3"/>
-      <limit effort="0" lower="-3.141" upper="1.308" velocity="3.054"/>
+      <origin xyz="0 0 0.9" rpy="0 0 0" />
+      <axis xyz="0 1 0" />
+      <parent link="${prefix}link_2" />
+      <child link="${prefix}link_3" />
+      <limit effort="0" lower="-3.141" upper="1.308" velocity="3.054" />
     </joint>
     <joint type="revolute" name="${prefix}joint_4">
-      <origin xyz="0 0 0.175" rpy="0 0 0"/>
-      <axis xyz="1 0 0"/>
-      <parent link="${prefix}link_3"/>
-      <child link="${prefix}link_4"/>
-      <limit effort="0" lower="-6.981" upper="6.981" velocity="4.363"/>
+      <origin xyz="0 0 0.175" rpy="0 0 0" />
+      <axis xyz="1 0 0" />
+      <parent link="${prefix}link_3" />
+      <child link="${prefix}link_4" />
+      <limit effort="0" lower="-6.981" upper="6.981" velocity="4.363" />
     </joint>
     <joint type="revolute" name="${prefix}joint_5">
-      <origin xyz="0.960 0 0 " rpy="0 0 0"/>
-      <axis xyz="0 1 0"/>
-      <parent link="${prefix}link_4"/>
-      <child link="${prefix}link_5"/>
-      <limit effort="0" lower="-2.181" upper="2.094" velocity="4.363"/>
+      <origin xyz="0.960 0 0 " rpy="0 0 0" />
+      <axis xyz="0 1 0" />
+      <parent link="${prefix}link_4" />
+      <child link="${prefix}link_5" />
+      <limit effort="0" lower="-2.181" upper="2.094" velocity="4.363" />
     </joint>
     <joint type="revolute" name="${prefix}joint_6">
-      <origin xyz="0.135 0 0 " rpy="0 0 0"/>
-      <axis xyz="1 0 0"/>
-      <parent link="${prefix}link_5"/>
-      <child link="${prefix}link_6"/>
-      <limit effort="0" lower="-6.981" upper="6.981" velocity="6.283"/>
+      <origin xyz="0.135 0 0 " rpy="0 0 0" />
+      <axis xyz="1 0 0" />
+      <parent link="${prefix}link_5" />
+      <child link="${prefix}link_6" />
+      <limit effort="0" lower="-6.981" upper="6.981" velocity="6.283" />
     </joint>
     <!-- end of joint list -->
@@ -200,14 +207,14 @@
     <link name="${prefix}base" />
     <joint name="${prefix}base_link-base" type="fixed">
-      <origin xyz="0 0 0" rpy="0 0 0"/>
-      <parent link="${prefix}base_link"/>
-      <child link="${prefix}base"/>
+      <origin xyz="0 0 0" rpy="0 0 0" />
+      <parent link="${prefix}base_link" />
+      <child link="${prefix}base" />
     </joint>
     <!-- ROS-Industrial 'flange' frame: attachment point for EEF models -->
-    <link name="${prefix}flange"/>
+    <link name="${prefix}flange" />
     <joint type="fixed" name="${prefix}joint_6-flange">
-      <origin xyz="0 0 0" rpy="0 0 0"/>
-      <parent link="${prefix}link_6"/>
-      <child link="${prefix}flange"/>
+      <origin xyz="0 0 0" rpy="0 0 0" />
+      <parent link="${prefix}link_6" />
+      <child link="${prefix}flange" />
     </joint>
     <!-- ROS-Industrial 'tool0' frame: all-zeros tool frame -->

Commit message: pow-76: update effort limits in abb robot xacro

File: abb_irb4600_support/urdf/irb4600_60_205_macro.urdf.xacro (robot description, xacro)
@@ -166,5 +166,5 @@
       <parent link="${prefix}base_link" />
       <child link="${prefix}link_1" />
-      <limit effort="0" lower="-3.141" upper="3.141" velocity="3.054" />
+      <limit effort="2000" lower="-3.141" upper="3.141" velocity="3.054" />
     </joint>
     <joint type="revolute" name="${prefix}joint_2">
@@ -173,5 +173,5 @@
       <parent link="${prefix}link_1" />
       <child link="${prefix}link_2" />
-      <limit effort="0" lower="-1.570" upper="2.617" velocity="3.054" />
+      <limit effort="5000" lower="-1.570" upper="2.617" velocity="3.054" />
     </joint>
     <joint type="revolute" name="${prefix}joint_3">
@@ -180,5 +180,5 @@
       <parent link="${prefix}link_2" />
       <child link="${prefix}link_3" />
-      <limit effort="0" lower="-3.141" upper="1.308" velocity="3.054" />
+      <limit effort="4000" lower="-3.141" upper="1.308" velocity="3.054" />
     </joint>
     <joint type="revolute" name="${prefix}joint_4">
@@ -187,5 +187,5 @@
       <parent link="${prefix}link_3" />
       <child link="${prefix}link_4" />
-      <limit effort="0" lower="-6.981" upper="6.981" velocity="4.363" />
+      <limit effort="1000" lower="-6.981" upper="6.981" velocity="4.363" />
     </joint>
     <joint type="revolute" name="${prefix}joint_5">
@@ -194,5 +194,5 @@
       <parent link="${prefix}link_4" />
       <child link="${prefix}link_5" />
-      <limit effort="0" lower="-2.181" upper="2.094" velocity="4.363" />
+      <limit effort="500" lower="-2.181" upper="2.094" velocity="4.363" />
     </joint>
     <joint type="revolute" name="${prefix}joint_6">
@@ -201,5 +201,5 @@
       <parent link="${prefix}link_5" />
       <child link="${prefix}link_6" />
-      <limit effort="0" lower="-6.981" upper="6.981" velocity="6.283" />
+      <limit effort="250" lower="-6.981" upper="6.981" velocity="6.283" />
     </joint>
     <!-- end of joint list -->
