Commit message: pow-76: add friction and damping to joints

File: abb_irb4600_support/urdf/irb4600_60_205_macro.urdf.xacro (robot description, xacro)
@@ -1,5 +1,6 @@
 <?xml version="1.0"?>
 <robot xmlns:xacro="http://ros.org/wiki/xacro">
-  <xacro:macro name="abb_irb4600_60_205" params="prefix:=''">
+  <xacro:macro name="abb_irb4600_60_205"
+    params="prefix:='' revolute_damping:=0 revolute_friction:=0">
     <!-- link list -->
     <link name="${prefix}base_link">
@@ -167,4 +168,5 @@
       <child link="${prefix}link_1" />
       <limit effort="2000" lower="-3.141" upper="3.141" velocity="3.054" />
+      <dynamics damping="${revolute_damping}" friction="${revolute_friction}" />
     </joint>
     <joint type="revolute" name="${prefix}joint_2">
@@ -174,4 +176,5 @@
       <child link="${prefix}link_2" />
       <limit effort="5000" lower="-1.570" upper="2.617" velocity="3.054" />
+      <dynamics damping="${revolute_damping}" friction="${revolute_friction}" />
     </joint>
     <joint type="revolute" name="${prefix}joint_3">
@@ -181,4 +184,5 @@
       <child link="${prefix}link_3" />
       <limit effort="4000" lower="-3.141" upper="1.308" velocity="3.054" />
+      <dynamics damping="${revolute_damping}" friction="${revolute_friction}" />
     </joint>
     <joint type="revolute" name="${prefix}joint_4">
@@ -188,4 +192,5 @@
       <child link="${prefix}link_4" />
       <limit effort="1000" lower="-6.981" upper="6.981" velocity="4.363" />
+      <dynamics damping="${revolute_damping}" friction="${revolute_friction}" />
     </joint>
     <joint type="revolute" name="${prefix}joint_5">
@@ -195,4 +200,5 @@
       <child link="${prefix}link_5" />
       <limit effort="500" lower="-2.181" upper="2.094" velocity="4.363" />
+      <dynamics damping="${revolute_damping}" friction="${revolute_friction}" />
     </joint>
     <joint type="revolute" name="${prefix}joint_6">
@@ -202,4 +208,5 @@
       <child link="${prefix}link_6" />
       <limit effort="250" lower="-6.981" upper="6.981" velocity="6.283" />
+      <dynamics damping="${revolute_damping}" friction="${revolute_friction}" />
     </joint>
     <!-- end of joint list -->

Commit message: make it possible to disable collision meshes

File: abb_irb4600_support/urdf/irb4600_60_205_macro.urdf.xacro (robot description, xacro)
@@ -2,12 +2,14 @@
 <robot xmlns:xacro="http://ros.org/wiki/xacro">
   <xacro:macro name="abb_irb4600_60_205"
-    params="prefix:='' revolute_damping:=0 revolute_friction:=0">
+    params="prefix:='' revolute_damping:=0 revolute_friction:=0 include_collision:=true">
     <!-- link list -->
     <link name="${prefix}base_link">
-      <collision name="collision">
-        <geometry>
-          <mesh filename="package://abb_irb4600_support/meshes/irb4600/collision/base_link.stl" />
-        </geometry>
-      </collision>
+      <xacro:if value="${include_collision}">
+        <collision name="collision">
+          <geometry>
+            <mesh filename="package://abb_irb4600_support/meshes/irb4600/collision/base_link.stl" />
+          </geometry>
+        </collision>
+      </xacro:if>
       <visual name="visual">
         <geometry>
@@ -29,9 +31,11 @@
     </link>
     <link name="${prefix}link_1">
-      <collision name="collision">
-        <geometry>
-          <mesh filename="package://abb_irb4600_support/meshes/irb4600/collision/link_1.stl" />
-        </geometry>
-      </collision>
+      <xacro:if value="${include_collision}">
+        <collision name="collision">
+          <geometry>
+            <mesh filename="package://abb_irb4600_support/meshes/irb4600/collision/link_1.stl" />
+          </geometry>
+        </collision>
+      </xacro:if>
       <visual name="visual">
         <geometry>
@@ -51,9 +55,11 @@
     </link>
     <link name="${prefix}link_2">
-      <collision name="collision">
-        <geometry>
-          <mesh filename="package://abb_irb4600_support/meshes/irb4600_60_205/collision/link_2.stl" />
-        </geometry>
-      </collision>
+      <xacro:if value="${include_collision}">
+        <collision name="collision">
+          <geometry>
+            <mesh filename="package://abb_irb4600_support/meshes/irb4600_60_205/collision/link_2.stl" />
+          </geometry>
+        </collision>
+      </xacro:if>
       <visual name="visual">
         <geometry>
@@ -73,9 +79,11 @@
     </link>
     <link name="${prefix}link_3">
-      <collision name="collision">
-        <geometry>
-          <mesh filename="package://abb_irb4600_support/meshes/irb4600_60_205/collision/link_3.stl" />
-        </geometry>
-      </collision>
+      <xacro:if value="${include_collision}">
+        <collision name="collision">
+          <geometry>
+            <mesh filename="package://abb_irb4600_support/meshes/irb4600_60_205/collision/link_3.stl" />
+          </geometry>
+        </collision>
+      </xacro:if>
       <visual name="visual">
         <geometry>
@@ -95,9 +103,11 @@
     </link>
     <link name="${prefix}link_4">
-      <collision name="collision">
-        <geometry>
-          <mesh filename="package://abb_irb4600_support/meshes/irb4600_60_205/collision/link_4.stl" />
-        </geometry>
-      </collision>
+      <xacro:if value="${include_collision}">
+        <collision name="collision">
+          <geometry>
+            <mesh filename="package://abb_irb4600_support/meshes/irb4600_60_205/collision/link_4.stl" />
+          </geometry>
+        </collision>
+      </xacro:if>
       <visual name="visual">
         <geometry>
@@ -117,9 +127,11 @@
     </link>
     <link name="${prefix}link_5">
-      <collision name="collision">
-        <geometry>
-          <mesh filename="package://abb_irb4600_support/meshes/irb4600_60_205/collision/link_5.stl" />
-        </geometry>
-      </collision>
+      <xacro:if value="${include_collision}">
+        <collision name="collision">
+          <geometry>
+            <mesh filename="package://abb_irb4600_support/meshes/irb4600_60_205/collision/link_5.stl" />
+          </geometry>
+        </collision>
+      </xacro:if>
       <visual name="visual">
         <geometry>
@@ -139,9 +151,11 @@
     </link>
     <link name="${prefix}link_6">
-      <collision name="collision">
-        <geometry>
-          <mesh filename="package://abb_irb4600_support/meshes/irb4600_60_205/collision/link_6.stl" />
-        </geometry>
-      </collision>
+      <xacro:if value="${include_collision}">
+        <collision name="collision">
+          <geometry>
+            <mesh filename="package://abb_irb4600_support/meshes/irb4600_60_205/collision/link_6.stl" />
+          </geometry>
+        </collision>
+      </xacro:if>
       <visual name="visual">
         <geometry>
